File: FlasherSplitter.kicad_pcb (KiCad board)
At the start: 2 copper layers, 0 parts

Commit message: Finish schematic and routing
Parts:
- added J1: 649012227222, Connectors:649012227222, F.Cu at (88.4, 98.2)
- added J2: 649006227222, Connectors:649006227222, F.Cu at (123.8, 106.7)
- added J3: 649006227222, Connectors:649006227222, F.Cu at (123.8, 90.3)
Routing:
- net Net-(J1-Pad1): track 0.00 -> 39.3 mm
- net Net-(J1-Pad7): track 0.00 -> 39.2 mm
- net Net-(J1-Pad3): track 0.00 -> 37.1 mm
- net Net-(J1-Pad6): track 0.00 -> 36.3 mm
- net Net-(J1-Pad8): track 0.00 -> 28.8 mm
- net Net-(J1-Pad5): track 0.00 -> 27.7 mm
- net Net-(J1-Pad2): track 0.00 -> 26.7 mm
- net Net-(J1-Pad4): track 0.00 -> 19.4 mm
- net Net-(J1-Pad12): track 0.00 -> 18.9 mm
- net Net-(J1-Pad9): track 0.00 -> 17.7 mm
- net Net-(J1-Pad10): track 0.00 -> 14.0 mm
- net Net-(J1-Pad11): track 0.00 -> 10.5 mm
Other:
- board outline added: 48.3 x 30.7 mm
