File: FlasherSplitter.sch (KiCad schematic (older format))
At the start: 0 parts

Commit message: Finish schematic and routing
Parts:
- added J1: 649012227222, Connectors:649012227222, symbol 649012227222
- added J2, J3: 649006227222, Connectors:649006227222, symbol 649006227222
Connections:
- new net: J1.7, J3.1
- new net: J1.8, J3.2
- new net: J1.9, J3.3
- new net: J1.10, J3.4
- new net: J1.11, J3.5
- new net: J1.12, J3.6
- new net: J1.1, J2.1
- new net: J1.2, J2.2
- new net: J1.3, J2.3
- new net: J1.4, J2.4
- new net: J1.5, J2.5
- new net: J1.6, J2.6
Changed lines of the file:
@@
 EESchema Schematic File Version 2
+LIBS:ADC
+LIBS:Amplifiers
+LIBS:Battery
+LIBS:Capacitors
+LIBS:Comparators
+LIBS:Connectors
+LIBS:Crystals
+LIBS:DAC
+LIBS:Diodes
+LIBS:Fuses
+LIBS:Inductors
+LIBS:Interface
+LIBS:Isolators
+LIBS:STMicroelectronics
+LIBS:PMIC
+LIBS:Power_Port
+LIBS:Relays
+LIBS:Resistors
+LIBS:Sensors
+LIBS:Switches
+LIBS:Transformers
+LIBS:Transistors
 LIBS:FlasherSplitter-cache
 EELAYER 26 0
@@
 Comment4 ""
 $EndDescr
+$Comp
+L 649006227222 J3
+U 1 1 5993713E
+P 6150 4050
+F 0 "J3" H 6150 4487 60  0000 C CNN
+F 1 "649006227222" H 6150 4381 60  0000 C CNN
+F 2 "Connectors:649006227222" H 6150 3150 60  0001 C CNN
+F 3 "http://katalog.we-online.de/em/datasheet/649006227222.pdf" H 6150 3050 60  0001 C CNN
+F 4 "Digikey" H 6150 3650 60  0001 C CNN "Supplier"
+F 5 "732-1939-ND" H 6150 3550 60  0001 C CNN "Supplier Part Number"
+F 6 "Wurth Electronics Inc." H 6150 3450 60  0001 C CNN "Manufacturer"
+F 7 "649006227222" H 6150 3350 60  0001 C CNN "Manufacturer Part Number"
+F 8 "HEADER MALE DUAL ANGLE W/MNT 6P" H 6150 3250 60  0001 C CNN "Description"
+	1    6150 4050
+	1    0    0    -1
+$EndComp
+$Comp
+L 649006227222 J2
+U 1 1 599372BE
+P 6150 3150
+F 0 "J2" H 6150 3587 60  0000 C CNN
+F 1 "649006227222" H 6150 3481 60  0000 C CNN
+F 2 "Connectors:649006227222" H 6150 2250 60  0001 C CNN
+F 3 "http://katalog.we-online.de/em/datasheet/649006227222.pdf" H 6150 2150 60  0001 C CNN
+F 4 "Digikey" H 6150 2750 60  0001 C CNN "Supplier"
+F 5 "732-1939-ND" H 6150 2650 60  0001 C CNN "Supplier Part Number"
+F 6 "Wurth Electronics Inc." H 6150 2550 60  0001 C CNN "Manufacturer"
+F 7 "649006227222" H 6150 2450 60  0001 C CNN "Manufacturer Part Number"
+F 8 "HEADER MALE DUAL ANGLE W/MNT 6P" H 6150 2350 60  0001 C CNN "Description"
+	1    6150 3150
+	1    0    0    -1
+$EndComp
+$Comp
+L 649012227222 J1
+U 1 1 599373EA
+P 5000 4150
+F 0 "J1" H 5056 5587 60  0000 C CNN
+F 1 "649012227222" H 5056 5481 60  0000 C CNN
+F 2 "Connectors:649012227222" H 5000 3250 60  0001 C CNN
+F 3 "http://katalog.we-online.de/em/datasheet/649012227222.pdf" H 5000 3150 60  0001 C CNN
+F 4 "Digikey" H 5000 3750 60  0001 C CNN "Supplier"
+F 5 "732-4771-ND" H 5000 3650 60  0001 C CNN "Supplier Part Number"
+F 6 "Wurth Electronics Inc." H 5000 3550 60  0001 C CNN "Manufacturer"
+F 7 "649012227222" H 5000 3450 60  0001 C CNN "Manufacturer Part Number"
+F 8 "HEADER MALE DUAL ANGLE W/MNT 12P" H 5000 3350 60  0001 C CNN "Description"
+	1    5000 4150
+	1    0    0    -1
+$EndComp
+Wire Wire Line
+	5150 2950 5750 2950
+Wire Wire Line
+	5750 2950 5750 2850
+Wire Wire Line
+	5750 2850 6500 2850
+Wire Wire Line
+	6500 2850 6500 3150
+Wire Wire Line
+	6500 3150 6350 3150
+Wire Wire Line
+	5150 3050 5750 3050
+Wire Wire Line
+	5750 3050 5750 3150
+Wire Wire Line
+	5750 3150 5950 3150
+Wire Wire Line
+	5150 3150 5700 3150
+Wire Wire Line
+	5700 3150 5700 3250
+Wire Wire Line
+	5700 3250 6400 3250
+Wire Wire Line
+	6400 3250 6400 3050
+Wire Wire Line
+	6400 3050 6350 3050
+Wire Wire Line
+	5150 3250 5650 3250
+Wire Wire Line
+	5650 3250 5650 3350
+Wire Wire Line
+	5650 3350 5900 3350
+Wire Wire Line
+	5900 3350 5900 3050
+Wire Wire Line
+	5900 3050 5950 3050
+Wire Wire Line
+	5150 3350 5600 3350
+Wire Wire Line
+	5600 3350 5600 3450
+Wire Wire Line
+	5600 3450 6450 3450
+Wire Wire Line
+	6450 3450 6450 2950
+Wire Wire Line
+	6450 2950 6350 2950
+Wire Wire Line
+	5150 3450 5550 3450
+Wire Wire Line
+	5550 3450 5550 3550
+Wire Wire Line
+	5550 3550 5800 3550
+Wire Wire Line
+	5800 3550 5800 2950
+Wire Wire Line
+	5800 2950 5950 2950
+Wire Wire Line
+	5150 3550 5500 3550
+Wire Wire Line
+	5500 3550 5500 3750
+Wire Wire Line
+	5500 3750 6500 3750
+Wire Wire Line
+	6500 3750 6500 4050
+Wire Wire Line
+	6500 4050 6350 4050
+Wire Wire Line
+	5150 3650 5450 3650
+Wire Wire Line
+	5450 3650 5450 4050
+Wire Wire Line
+	5450 4050 5950 4050
+Wire Wire Line
+	5150 3750 5400 3750
+Wire Wire Line
+	5400 3750 5400 4150
+Wire Wire Line
+	5400 4150 6400 4150
+Wire Wire Line
+	6400 4150 6400 3950
+Wire Wire Line
+	6400 3950 6350 3950
+Wire Wire Line
+	5150 3850 5500 3850
+Wire Wire Line
+	5500 3850 5500 3950
+Wire Wire Line
+	5500 3950 5950 3950
+Wire Wire Line
+	5150 3950 5350 3950
+Wire Wire Line
+	5350 3950 5350 4250
+Wire Wire Line
+	5350 4250 6450 4250
+Wire Wire Line
+	6450 4250 6450 3850
+Wire Wire Line
+	6450 3850 6350 3850
+Wire Wire Line
+	5150 4050 5300 4050
+Wire Wire Line
+	5300 4050 5300 4350
+Wire Wire Line
+	5300 4350 5900 4350
+Wire Wire Line
+	5900 4350 5900 3850
+Wire Wire Line
+	5900 3850 5950 3850
 $EndSCHEMATC
